Commit message: add joint plugins for GazeboSim

File: baxter_description/urdf/baxter.urdf (robot description, URDF)
Before this commit: robot baxter, 57 links, 56 joints
Links:
- link head: geometry collision sphere radius=0.001; visual mesh filename=file:///home/olivier/code/libs/ros2/install/baxter_descript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
- link left_lower_elbow: geometry collision cylinder length=0.10 radius=0.06; visual mesh filename=file:///home/olivier/code/libs/ros2/install/baxter_descript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
- link left_lower_forearm: geometry collision cylinder length=0.10 radius=0.06; visual mesh filename=file:///home/olivier/code/libs/ros2/install/baxter_descript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
- link left_lower_shoulder: geometry collision cylinder length=0.12 radius=0.06; visual mesh filename=file:///home/olivier/code/libs/ros2/install/baxter_descript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
- link left_upper_elbow: geometry collision cylinder length=0.107 radius=0.06; visual mesh filename=file:///home/olivier/code/libs/ros2/install/baxter_descript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
- link left_upper_forearm: geometry collision cylinder length=0.088 radius=0.06; visual mesh filename=file:///home/olivier/code/libs/ros2/install/baxter_descript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
- link left_upper_shoulder: geometry collision cylinder length=0.2722 radius=0.06; visual mesh filename=file:///home/olivier/code/libs/ros2/install/baxter_descript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
- link left_wrist: geometry collision cylinder length=0.165 radius=0.06; visual mesh filename=file:///home/olivier/code/libs/ros2/install/baxter_descript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
- link pedestal: geometry collision mesh filename=file:///home/olivier/code/libs/ros2/install/baxter_descript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; visual mesh filename=file:///home/olivier/code/libs/ros2/install/baxter_descript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
- link right_lower_elbow: geometry collision cylinder length=0.10 radius=0.06; visual mesh filename=file:///home/olivier/code/libs/ros2/install/baxter_descript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
- link right_lower_forearm: geometry collision cylinder length=0.10 radius=0.06; visual mesh filename=file:///home/olivier/code/libs/ros2/install/baxter_descript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
- link right_lower_shoulder: geometry collision cylinder length=0.12 radius=0.06; visual mesh filename=file:///home/olivier/code/libs/ros2/install/baxter_descript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
- link right_upper_elbow: geometry collision cylinder length=0.107 radius=0.06; visual mesh filename=file:///home/olivier/code/libs/ros2/install/baxter_descript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
- link right_upper_forearm: geometry collision cylinder length=0.088 radius=0.06; visual mesh filename=file:///home/olivier/code/libs/ros2/install/baxter_descript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
- link right_upper_shoulder: geometry collision cylinder length=0.2722 radius=0.06; visual mesh filename=file:///home/olivier/code/libs/ros2/install/baxter_descript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
- link right_wrist: geometry collision cylinder length=0.165 radius=0.06; visual mesh filename=file:///home/olivier/code/libs/ros2/install/baxter_descript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
- link screen: geometry collision sphere radius=0.001; visual mesh filename=file:///home/olivier/code/libs/ros2/install/baxter_descript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
- link torso: geometry collision mesh filename=file:///home/olivier/code/libs/ros2/install/baxter_descript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; visual mesh filename=file:///home/olivier/code/libs/ros2/install/baxter_descript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
Joints:
- joint l_gripper_l_finger_joint: origin xyz=0.0 -0.0015 0.02 rpy=0 0 0 -> xyz=0.0 -0.0014999999999999996 0.02 rpy=0 0 0
- joint l_gripper_r_finger_joint: origin xyz=0.0 0.0015 0.02 rpy=0 0 0 -> xyz=0.0 0.0014999999999999996 0.02 rpy=0 0 0
- joint left_endpoint: origin xyz=0 0 0.1327 rpy=0 0 0 -> xyz=0 0 0.13269999999999998 rpy=0 0 0
- joint r_gripper_l_finger_joint: origin xyz=0.0 -0.0015 0.02 rpy=0 0 0 -> xyz=0.0 -0.0014999999999999996 0.02 rpy=0 0 0
- joint r_gripper_r_finger_joint: origin xyz=0.0 0.0015 0.02 rpy=0 0 0 -> xyz=0.0 0.0014999999999999996 0.02 rpy=0 0 0
- joint right_endpoint: origin xyz=0 0 0.1327 rpy=0 0 0 -> xyz=0 0 0.13269999999999998 rpy=0 0 0

File: baxter_description/urdf/baxter.urdf.xacro (robot description, xacro)
@@ -17,3 +17,5 @@
   <!-- Right End Effector -->
   <xacro:include filename="$(find baxter_description)/urdf/right_end_effector.urdf.xacro" />
+  <!-- Gazebo plugins -->
+  <xacro:include filename="$(find baxter_description)/urdf/gazebosim.urdf.xacro" />
 </robot>

File: baxter_description/urdf/baxter_base/baxter_base.urdf.xacro (robot description, xacro)
@@ -12,5 +12,5 @@
       <origin rpy="0 0 0" xyz="0 0 0"/>
       <geometry>
-        <mesh filename="package://baxter_description/meshes/torso/base_link.DAE"/>
+        <mesh filename="file://$(find baxter_description)/meshes/torso/base_link.DAE"/>
       </geometry>
       <material name="darkgray">
@@ -21,5 +21,5 @@
       <origin rpy="0 0 0" xyz="0 0 0"/>
       <geometry>
-        <mesh filename="package://baxter_description/meshes/torso/base_link_collision.DAE"/>
+        <mesh filename="file://$(find baxter_description)/meshes/torso/base_link_collision.DAE"/>
       </geometry>
     </collision>
@@ -48,5 +48,5 @@
       <origin rpy="0 0 0" xyz="0 0 .00953"/>
       <geometry>
-        <mesh filename="package://baxter_description/meshes/head/H0.DAE"/>
+        <mesh filename="file://$(find baxter_description)/meshes/head/H0.DAE"/>
       </geometry>
       <material name="darkgray">
@@ -92,5 +92,5 @@
       <origin rpy="0 -1.57079632679 0" xyz="0 -.00953 -.0347"/>
       <geometry>
-        <mesh filename="package://baxter_description/meshes/head/H1.DAE"/>
+        <mesh filename="file://$(find baxter_description)/meshes/head/H1.DAE"/>
       </geometry>
       <material name="darkred">
@@ -256,5 +256,5 @@
       <origin rpy="0 0 0" xyz="0 0 0"/>
       <geometry>
-        <mesh filename="package://baxter_description/meshes/upper_shoulder/S0.DAE"/>
+        <mesh filename="file://$(find baxter_description)/meshes/upper_shoulder/S0.DAE"/>
       </geometry>
       <material name="darkred">
@@ -278,5 +278,5 @@
       <origin rpy="0 0 0" xyz="0 0 0"/>
       <geometry>
-        <mesh filename="package://baxter_description/meshes/lower_shoulder/S1.DAE"/>
+        <mesh filename="file://$(find baxter_description)/meshes/lower_shoulder/S1.DAE"/>
       </geometry>
       <material name="darkred">
@@ -300,5 +300,5 @@
       <origin rpy="0 0 0" xyz="0 0 0"/>
       <geometry>
-        <mesh filename="package://baxter_description/meshes/upper_elbow/E0.DAE"/>
+        <mesh filename="file://$(find baxter_description)/meshes/upper_elbow/E0.DAE"/>
       </geometry>
       <material name="darkred">
@@ -335,5 +335,5 @@
       <origin rpy="0 0 0" xyz="0 0 0"/>
       <geometry>
-        <mesh filename="package://baxter_description/meshes/lower_elbow/E1.DAE"/>
+        <mesh filename="file://$(find baxter_description)/meshes/lower_elbow/E1.DAE"/>
       </geometry>
       <material name="darkred">
@@ -357,5 +357,5 @@
       <origin rpy="0 0 0" xyz="0 0 0"/>
       <geometry>
-        <mesh filename="package://baxter_description/meshes/upper_forearm/W0.DAE"/>
+        <mesh filename="file://$(find baxter_description)/meshes/upper_forearm/W0.DAE"/>
       </geometry>
       <material name="darkred">
@@ -399,5 +399,5 @@
       <origin rpy="0 0 0" xyz="0 0 0"/>
       <geometry>
-        <mesh filename="package://baxter_description/meshes/lower_forearm/W1.DAE"/>
+        <mesh filename="file://$(find baxter_description)/meshes/lower_forearm/W1.DAE"/>
       </geometry>
       <material name="darkred">
@@ -421,5 +421,5 @@
       <origin rpy="0 0 0" xyz="0 0 0"/>
       <geometry>
-        <mesh filename="package://baxter_description/meshes/wrist/W2.DAE"/>
+        <mesh filename="file://$(find baxter_description)/meshes/wrist/W2.DAE"/>
       </geometry>
       <material name="lightgrey">
@@ -624,5 +624,5 @@
       <origin rpy="0 0 0" xyz="0 0 0"/>
       <geometry>
-        <mesh filename="package://baxter_description/meshes/upper_shoulder/S0.DAE"/>
+        <mesh filename="file://$(find baxter_description)/meshes/upper_shoulder/S0.DAE"/>
       </geometry>
       <material name="darkred">
@@ -646,5 +646,5 @@
       <origin rpy="0 0 0" xyz="0 0 0"/>
       <geometry>
-        <mesh filename="package://baxter_description/meshes/lower_shoulder/S1.DAE"/>
+        <mesh filename="file://$(find baxter_description)/meshes/lower_shoulder/S1.DAE"/>
       </geometry>
       <material name="darkred">
@@ -668,5 +668,5 @@
       <origin rpy="0 0 0" xyz="0 0 0"/>
       <geometry>
-        <mesh filename="package://baxter_description/meshes/upper_elbow/E0.DAE"/>
+        <mesh filename="file://$(find baxter_description)/meshes/upper_elbow/E0.DAE"/>
       </geometry>
       <material name="darkred">
@@ -703,5 +703,5 @@
       <origin rpy="0 0 0" xyz="0 0 0"/>
       <geometry>
-        <mesh filename="package://baxter_description/meshes/lower_elbow/E1.DAE"/>
+        <mesh filename="file://$(find baxter_description)/meshes/lower_elbow/E1.DAE"/>
       </geometry>
       <material name="darkred">
@@ -725,5 +725,5 @@
       <origin rpy="0 0 0" xyz="0 0 0"/>
       <geometry>
-        <mesh filename="package://baxter_description/meshes/upper_forearm/W0.DAE"/>
+        <mesh filename="file://$(find baxter_description)/meshes/upper_forearm/W0.DAE"/>
       </geometry>
       <material name="darkred">
@@ -767,5 +767,5 @@
       <origin rpy="0 0 0" xyz="0 0 0"/>
       <geometry>
-        <mesh filename="package://baxter_description/meshes/lower_forearm/W1.DAE"/>
+        <mesh filename="file://$(find baxter_description)/meshes/lower_forearm/W1.DAE"/>
       </geometry>
       <material name="darkred">
@@ -789,5 +789,5 @@
       <origin rpy="0 0 0" xyz="0 0 0"/>
       <geometry>
-        <mesh filename="package://baxter_description/meshes/wrist/W2.DAE"/>
+        <mesh filename="file://$(find baxter_description)/meshes/wrist/W2.DAE"/>
       </geometry>
       <material name="lightgrey">

File: baxter_description/urdf/pedestal/pedestal.xacro (robot description, xacro)
@@ -7,5 +7,5 @@
       <origin rpy="0 0 0" xyz="0 0 0"/>
       <geometry>
-        <mesh filename="package://baxter_description/meshes/base/PEDESTAL.DAE"/>
+        <mesh filename="file://$(find baxter_description)/meshes/base/PEDESTAL.DAE"/>
       </geometry>
       <material name="darkgray">
@@ -16,5 +16,5 @@
       <origin rpy="0 0 0" xyz="0 0 0"/>
       <geometry>
-        <mesh filename="package://baxter_description/meshes/base/pedestal_link_collision.DAE"/>
+        <mesh filename="file://$(find baxter_description)/meshes/base/pedestal_link_collision.DAE"/>
       </geometry>
     </collision>

File: rethink_ee_description/urdf/electric_gripper/rethink_electric_gripper.xacro (robot description, xacro)
@@ -8,5 +8,5 @@
         <origin rpy="${-pi/2} ${pi} 0" xyz="0 0 0"/>
         <geometry>
-          <mesh filename="package://rethink_ee_description/meshes/electric_gripper/electric_gripper_base.DAE"/>
+          <mesh filename="file://$(find rethink_ee_description)/meshes/electric_gripper/electric_gripper_base.DAE"/>
         </geometry>
       </visual>
