Commit message: gz plugins robust to Jetty

File: baxter_description/urdf/baxter.urdf.xacro (robot description, xacro)
@@ -5,12 +5,8 @@
   <xacro:property name="PI" value="3.1415927"/>
   <!-- Baxter Base URDF -->
-  <xacro:include filename="$(find baxter_description)/urdf/baxter_base/baxter_base.urdf.xacro">
-<!--     <xacro:arg name="gazebo" value="$(arg gazebo)"/> -->
-  </xacro:include>
+  <xacro:include filename="$(find baxter_description)/urdf/baxter_base/baxter_base.urdf.xacro"/>
   <!-- Baxter Pedestal -->
   <xacro:if value="$(arg pedestal)">
-    <xacro:include filename="$(find baxter_description)/urdf/pedestal/pedestal.xacro">
-<!--       <xacro:arg name="gazebo" value="$(arg gazebo)"/> -->
-    </xacro:include>
+    <xacro:include filename="$(find baxter_description)/urdf/pedestal/pedestal.xacro"/>
   </xacro:if>
   <!-- Left End Effector -->
@@ -19,4 +15,6 @@
   <xacro:include filename="$(find baxter_description)/urdf/right_end_effector.urdf.xacro" />
   <!-- Gazebo plugins -->
+  <xacro:if value="$(arg gazebo)">
   <xacro:include filename="$(find baxter_description)/urdf/gazebosim.urdf.xacro" />
+</xacro:if>
 </robot>

File: baxter_description/urdf/baxter_base/baxter_base.urdf.xacro (robot description, xacro)
@@ -1,43 +1,4 @@
 <?xml version="1.0" ?>
 <robot name="baxter" xmlns:xacro="http://www.ros.org/wiki/xacro">
-<!--  <xacro:if value="$(arg gazebo)">
-    <xacro:property name="mass_scale" value=".1"/>
-    <xacro:include filename="$(find baxter_description)/urdf/baxter_base/baxter_base.gazebo.xacro" />
-  </xacro:if>
-  <xacro:unless value="$(arg gazebo)">
-    <xacro:property name="mass_scale" value=".1"/>
-  </xacro:unless>-->
-  <xacro:macro name="range_sensor" params="side">
- <!-- <gazebo>
-  <sensor name="range_${side}" type="gpu_lidar">
-    <pose >1 0 0 0 ${PI/2} 0</pose>
-    <topic>${side}_range</topic>
-    <update_rate>10</update_rate>
-    <ray>
-        <scan>
-<horizontal>
-                <samples>10</samples>
-                <resolution>1</resolution>
-                <min_angle>-1.396263</min_angle>
-                <max_angle>1.396263</max_angle>
-            </horizontal>
-            <vertical>
-                <samples>1</samples>
-                <resolution>0.01</resolution>
-                <min_angle>0</min_angle>
-                <max_angle>0</max_angle>
-            </vertical>
-        </scan>
-        <range>
-            <min>0.1</min>
-            <max>1.</max>
-            <resolution>0.01</resolution>
-        </range>
-    </ray>
-    <always_on>1</always_on>
-    <visualize>true</visualize>
-</sensor>
-</gazebo>-->
-</xacro:macro>
   <link name="base">
   </link>
@@ -524,5 +485,4 @@
       <inertia ixx="1e-08" ixy="0" ixz="0" iyy="1e-08" iyz="0" izz="1e-08"/>
     </inertial>
-    <xacro:range_sensor side="right"/>
   </link>
   <link name="right_hand_accelerometer">
@@ -909,5 +869,4 @@
       <inertia ixx="1e-08" ixy="0" ixz="0" iyy="1e-08" iyz="0" izz="1e-08"/>
     </inertial>
-    <xacro:range_sensor side="left"/>
   </link>
   <joint name="left_torso_arm_mount" type="fixed">

File: baxter_description/urdf/gazebosim.urdf.xacro (robot description, xacro)
@@ -5,5 +5,5 @@
        <gazebo>
         <!-- Velocity control -->
-        <plugin filename="libignition-gazebo-joint-controller-system.so" name="ignition::gazebo::systems::JointController">
+        <plugin filename="ignition-gazebo-joint-controller-system" name="ignition::gazebo::systems::JointController">
             <joint_name>${joint}</joint_name>
             <topic>${joint}_cmd_vel</topic>
@@ -80,5 +80,5 @@
 </xacro:macro>
     <gazebo>
-        <plugin filename="libignition-gazebo-joint-state-publisher-system.so" name="ignition::gazebo::systems::JointStatePublisher"/>
+        <plugin filename="ignition-gazebo-joint-state-publisher-system" name="ignition::gazebo::systems::JointStatePublisher"/>
 </gazebo>
         <xacro:arm_plugins side="left"/>
