Commit message: embed headers for ROS 1 Baxter msgs to avoid having to locate them

File: baxter_description/urdf/gazebosim.urdf.xacro (robot description, xacro)
@@ -7,12 +7,49 @@
             <p_gain>10.</p_gain>
             <i_gain>1.</i_gain>
-            <d_gain>0.1</d_gain>
+            <d_gain>1.</d_gain>
+            <i_max>100</i_max>
+            <i_min>-100</i_min>
         </plugin>
         <!-- Velocity control -->
-        <plugin filename="libignition-gazebo-joint-controller-system.so"
-        name="ignition::gazebo::systems::JointController">
+<!--        <plugin filename="libignition-gazebo-joint-controller-system.so" name="ignition::gazebo::systems::JointController">
             <joint_name>${joint}</joint_name>
-        </plugin>
+            <topic>${joint}_cmd_vel</topic>
+        </plugin>  -->
      </xacro:macro>
+     <xacro:macro name="camera_plugin" params="link">
+        <gazebo reference="${link}">
+         <sensor name="${link}" type="camera">
+          <camera>
+            <horizontal_fov>1.047</horizontal_fov> -->
+            <image>
+              <width>640</width>
+              <height>400</height>
+            </image>
+            <clip>
+              <near>0.1</near>
+              <far>100</far>
+            </clip>
+          </camera>
+          <always_on>1</always_on>
+          <update_rate>30</update_rate>
+          <visualize>true</visualize>
+          <topic>${link}</topic>
+          <enable_metrics>false</enable_metrics>
+        </sensor>
+<!--        <plugin filename="ImageDisplay" name="Image Display">
+        <ignition-gui>
+          <title>RGB camera</title>
+          <property key="state" type="string" name="dummy">floating</property>
+          <property type="double" key="width" name="dummy">350</property>
+          <property type="double" key="height" name="dummy">315</property>
+        </ignition-gui>
+        <topic>${link}_image</topic>
+        <topic_picker>false</topic_picker>
+      </plugin>-->
+    </gazebo>
+    </xacro:macro>
+     <xacro:macro name="range" params="link">
+        <!-- Not supported -->
+    </xacro:macro>
     <gazebo>
         <plugin filename="libignition-gazebo-joint-state-publisher-system.so" name="ignition::gazebo::systems::JointStatePublisher"/>
@@ -32,4 +69,9 @@
         <xacro:joint_controller joint="left_w1"/>
         <xacro:joint_controller joint="left_w2"/>
+        <xacro:range link="left_hand_range"/>
+        <xacro:range link="right_hand_range"/>
     </gazebo>
+<!--         <xacro:camera_plugin link="head_camera"/> -->
+        <xacro:camera_plugin link="left_hand_camera"/>
+<!--         <xacro:camera_plugin link="right_hand_camera_axis"/> -->
 </robot>

Commit message: with camera_gz axis

File: baxter_description/urdf/gazebosim.urdf.xacro (robot description, xacro)
@@ -31,5 +31,11 @@
         <xacro:joint_controller joint="${side}_w1" cmd_max="15" p="900" i=".1" d=".01"/>
         <xacro:joint_controller joint="${side}_w2" cmd_max="15" p="1000" i=".01" d=".01"/>
-        <gazebo reference="${side}_hand_camera_axis">
+        <link name="${side}_hand_camera_gz"/>
+        <joint name="${side}_camera" type="fixed">
+          <parent link="${side}_hand_camera_axis"/>
+          <child link="${side}_hand_camera_gz"/>
+          <origin rpy="0 ${-PI/2} 0"/>
+        </joint>
+        <gazebo reference="${side}_hand_camera_gz">
          <sensor name="${side}_camera" type="camera">
           <camera>
