Commit message: cameras + range sensors in Gazebo

File: baxter_description/urdf/baxter_base/baxter_base.urdf.xacro (robot description, xacro)
@@ -8,4 +8,36 @@
     <xacro:property name="mass_scale" value=".1"/>
   </xacro:unless>-->
+  <xacro:macro name="range_sensor" params="side">
+ <!-- <gazebo>
+  <sensor name="range_${side}" type="gpu_lidar">
+    <pose >1 0 0 0 ${PI/2} 0</pose>
+    <topic>${side}_range</topic>
+    <update_rate>10</update_rate>
+    <ray>
+        <scan>
+<horizontal>
+                <samples>10</samples>
+                <resolution>1</resolution>
+                <min_angle>-1.396263</min_angle>
+                <max_angle>1.396263</max_angle>
+            </horizontal>
+            <vertical>
+                <samples>1</samples>
+                <resolution>0.01</resolution>
+                <min_angle>0</min_angle>
+                <max_angle>0</max_angle>
+            </vertical>
+        </scan>
+        <range>
+            <min>0.1</min>
+            <max>1.</max>
+            <resolution>0.01</resolution>
+        </range>
+    </ray>
+    <always_on>1</always_on>
+    <visualize>true</visualize>
+</sensor>
+</gazebo>-->
+</xacro:macro>
   <link name="base">
   </link>
@@ -492,4 +524,5 @@
       <inertia ixx="1e-08" ixy="0" ixz="0" iyy="1e-08" iyz="0" izz="1e-08"/>
     </inertial>
+    <xacro:range_sensor side="right"/>
   </link>
   <link name="right_hand_accelerometer">
@@ -876,4 +909,5 @@
       <inertia ixx="1e-08" ixy="0" ixz="0" iyy="1e-08" iyz="0" izz="1e-08"/>
     </inertial>
+    <xacro:range_sensor side="left"/>
   </link>
   <joint name="left_torso_arm_mount" type="fixed">

File: baxter_description/urdf/gazebosim.urdf.xacro (robot description, xacro)
@@ -21,9 +21,18 @@
         </plugin>-->
      </xacro:macro>
-     <xacro:macro name="camera_plugin" params="link">
-        <gazebo reference="${link}">
-         <sensor name="${link}" type="camera">
+    <xacro:macro name="arm_plugins" params="side">
+        <!-- gains from baxter_sim_hardware
+      https://github.com/RethinkRobotics/baxter_simulator/blob/master/baxter_sim_hardware/config/baxter_sim_controllers.yaml -->
+        <xacro:joint_controller joint="${side}_s0" cmd_max="50" p="700" i="0.01" d="10"/>
+        <xacro:joint_controller joint="${side}_s1" cmd_max="50" p="10000" i="10" d="10"/>
+        <xacro:joint_controller joint="${side}_e0" cmd_max="50" p="4500" i="35" d="1"/>
+        <xacro:joint_controller joint="${side}_e1" cmd_max="50" p="5500" i="60" d="2"/>
+        <xacro:joint_controller joint="${side}_w0" cmd_max="15" p="1000" i="30" d="0.01"/>
+        <xacro:joint_controller joint="${side}_w1" cmd_max="15" p="900" i=".1" d=".01"/>
+        <xacro:joint_controller joint="${side}_w2" cmd_max="15" p="1000" i=".01" d=".01"/>
+        <gazebo reference="${side}_hand_camera_axis">
+         <sensor name="${side}_camera" type="camera">
           <camera>
-            <horizontal_fov>1.047</horizontal_fov> -->
+            <horizontal_fov>1.047</horizontal_fov>
             <image>
               <width>640</width>
@@ -37,36 +46,13 @@
           <always_on>1</always_on>
           <update_rate>30</update_rate>
-          <visualize>true</visualize>
-          <topic>${link}</topic>
-          <enable_metrics>false</enable_metrics>
+          <visualize>false</visualize>
+          <topic>${side}_arm/image</topic>
         </sensor>
-<!--        <plugin filename="ImageDisplay" name="Image Display">
-        <ignition-gui>
-          <title>RGB camera</title>
-          <property key="state" type="string" name="dummy">floating</property>
-          <property type="double" key="width" name="dummy">350</property>
-          <property type="double" key="height" name="dummy">315</property>
-        </ignition-gui>
-        <topic>${link}_image</topic>
-        <topic_picker>false</topic_picker>
-      </plugin>-->
-    </gazebo>
-    </xacro:macro>
-    <xacro:macro name="arm_plugins" params="side">
-        <!-- gains from baxter_sim_hardware
-      https://github.com/RethinkRobotics/baxter_simulator/blob/master/baxter_sim_hardware/config/baxter_sim_controllers.yaml -->
-        <xacro:joint_controller joint="${side}_s0" cmd_max="50" p="700" i="0.01" d="10"/>
-        <xacro:joint_controller joint="${side}_s1" cmd_max="50" p="10000" i="10" d="10"/>
-        <xacro:joint_controller joint="${side}_e0" cmd_max="50" p="4500" i="35" d="1"/>
-        <xacro:joint_controller joint="${side}_e1" cmd_max="50" p="5500" i="60" d="2"/>
-        <xacro:joint_controller joint="${side}_w0" cmd_max="15" p="1000" i="30" d="0.01"/>
-        <xacro:joint_controller joint="${side}_w1" cmd_max="15" p="900" i=".1" d=".01"/>
-        <xacro:joint_controller joint="${side}_w2" cmd_max="15" p="1000" i=".01" d=".01"/>
-        <xacro:camera_plugin link="${side}_hand_camera"/>
+      </gazebo>
   <gazebo reference="${side}_hand_range">
   <sensor name="range_${side}" type="gpu_lidar">
-<!--     <pose relative_to="${side}_hand_range">0 0 0 0 ${PI/2} 0</pose> -->
-    <pose >0 0 0 0 ${PI/2} 0</pose>
-    <topic>${side}_range</topic>
+<!--     <pose relative_to="${side}_hand_range">0 0 0 ${PI/2} 0 0</pose> -->
+<!--     <pose >1 1 1 0 ${PI/2} 0</pose> -->
+    <topic>${side}_arm/range</topic>
     <update_rate>10</update_rate>
     <ray>
@@ -75,17 +61,17 @@
                 <samples>10</samples>
                 <resolution>1</resolution>
-                <min_angle>-1.396263</min_angle>
-                <max_angle>1.396263</max_angle>
+                <min_angle>-0.3</min_angle>
+                <max_angle>0.3</max_angle>
             </horizontal>
             <vertical>
-                <samples>1</samples>
-                <resolution>0.01</resolution>
-                <min_angle>0</min_angle>
-                <max_angle>0</max_angle>
+                <samples>10</samples>
+                <resolution>1</resolution>
+                <min_angle>-0.3</min_angle>
+                <max_angle>0.3</max_angle>
             </vertical>
         </scan>
         <range>
-            <min>0.1</min>
-            <max>1.</max>
+            <min>0.15</min>
+            <max>0.5</max>
             <resolution>0.01</resolution>
         </range>
@@ -95,5 +81,5 @@
 </sensor>
 </gazebo>
-     </xacro:macro>
+</xacro:macro>
     <gazebo>
         <plugin filename="libignition-gazebo-joint-state-publisher-system.so" name="ignition::gazebo::systems::JointStatePublisher"/>

Commit message: do not force node name in bridge

File: baxter_description/urdf/baxter_base/baxter_base.urdf.xacro (robot description, xacro)
@@ -262,5 +262,5 @@
     <child link="screen"/>
   </joint>
-  <joint name="head_camera" type="fixed">
+  <joint name="head_camera_fixed" type="fixed">
     <origin rpy="1.75057 0 1.57079632679" xyz="0.12839 0 0.06368"/>
     <parent link="head"/>
@@ -621,5 +621,5 @@
     <dynamics damping="0.7" friction="0.0"/>
   </joint>
-  <joint name="right_hand" type="fixed">
+  <joint name="right_hand_fixed" type="fixed">
     <origin rpy="0 0 0" xyz="0 0 0.11355"/>
     <axis xyz="0 0 1"/>
@@ -627,20 +627,20 @@
     <child link="right_hand"/>
   </joint>
-  <joint name="right_hand_camera" type="fixed">
+  <joint name="right_hand_camera_fixed" type="fixed">
     <origin rpy="0 0 -1.57079633" xyz="0.03825 0.012 0.015355"/>
     <parent link="right_hand"/>
     <child link="right_hand_camera"/>
   </joint>
-  <joint name="right_hand_camera_axis" type="fixed">
+  <joint name="right_hand_camera_axis_fixed" type="fixed">
     <origin rpy="0 0 0" xyz="0.03825 0.012 0.015355"/>
     <parent link="right_hand"/>
     <child link="right_hand_camera_axis"/>
   </joint>
-  <joint name="right_hand_range" type="fixed">
+  <joint name="right_hand_range_fixed" type="fixed">
     <origin rpy="0 -1.57079632679 -1.57079632679" xyz="0.032 -0.020245 0.0288"/>
     <parent link="right_hand"/>
     <child link="right_hand_range"/>
   </joint>
-  <joint name="right_hand_accelerometer" type="fixed">
+  <joint name="right_hand_accelerometer_fixed" type="fixed">
     <origin rpy="0 0 0" xyz="0.00198 0.000133 -0.0146"/>
     <parent link="right_hand"/>
@@ -990,5 +990,5 @@
     <dynamics damping="0.7" friction="0.0"/>
   </joint>
-  <joint name="left_hand" type="fixed">
+  <joint name="left_hand_fixed" type="fixed">
     <origin rpy="0 0 0" xyz="0 0 0.11355"/>
     <axis xyz="0 0 1"/>
@@ -996,20 +996,20 @@
     <child link="left_hand"/>
   </joint>
-  <joint name="left_hand_camera" type="fixed">
+  <joint name="left_hand_camera_fixed" type="fixed">
     <origin rpy="0 0 -1.57079633" xyz="0.03825 0.012 0.015355"/>
     <parent link="left_hand"/>
     <child link="left_hand_camera"/>
   </joint>
-  <joint name="left_hand_camera_axis" type="fixed">
+  <joint name="left_hand_camera_axis_fixed" type="fixed">
     <origin rpy="0 0 0" xyz="0.03825 0.012 0.015355"/>
     <parent link="left_hand"/>
     <child link="left_hand_camera_axis"/>
   </joint>
-  <joint name="left_hand_range" type="fixed">
+  <joint name="left_hand_range_fixed" type="fixed">
     <origin rpy="0 -1.57079632679 -1.57079632679" xyz="0.032 -0.020245 0.0288"/>
     <parent link="left_hand"/>
     <child link="left_hand_range"/>
   </joint>
-  <joint name="left_hand_accelerometer" type="fixed">
+  <joint name="left_hand_accelerometer_fixed" type="fixed">
     <origin rpy="0 0 0" xyz="0.00198 0.000133 -0.0146"/>
     <parent link="left_hand"/>

File: rethink_ee_description/urdf/electric_gripper/fingers/basic_hard_tip.xacro (robot description, xacro)
@@ -10,5 +10,5 @@
         <origin rpy="0 0 ${pi*(g_reflect+1)/2}" xyz="0 0 0"/>
         <geometry>
-          <mesh filename="package://rethink_ee_description/meshes/electric_gripper/fingers/basic_hard_tip.DAE" />
+          <mesh filename="file://$(find rethink_ee_description)/meshes/electric_gripper/fingers/basic_hard_tip.DAE" />
         </geometry>
       </visual>

File: rethink_ee_description/urdf/electric_gripper/fingers/basic_soft_tip.xacro (robot description, xacro)
@@ -10,5 +10,5 @@
         <origin rpy="0 0 ${pi*(g_reflect+1)/2}" xyz="0 0 0"/>
         <geometry>
-          <mesh filename="package://rethink_ee_description/meshes/electric_gripper/fingers/basic_soft_tip.DAE" />
+          <mesh filename="file://$(find rethink_ee_description)/meshes/electric_gripper/fingers/basic_soft_tip.DAE" />
         </geometry>
       </visual>

File: rethink_ee_description/urdf/electric_gripper/fingers/extended_narrow.xacro (robot description, xacro)
@@ -8,5 +8,5 @@
         <origin rpy="0 0 ${-pi/2*(reflect+1)}" xyz="0 0 0"/>
         <geometry>
-          <mesh filename="package://rethink_ee_description/meshes/electric_gripper/fingers/extended_narrow.DAE" />
+          <mesh filename="file://$(find rethink_ee_description)/meshes/electric_gripper/fingers/extended_narrow.DAE" />
         </geometry>
       </visual>

File: rethink_ee_description/urdf/electric_gripper/fingers/extended_wide.xacro (robot description, xacro)
@@ -8,5 +8,5 @@
         <origin rpy="0 0 ${-pi/2*(reflect+1)}" xyz="0 0 0"/>
         <geometry>
-          <mesh filename="package://rethink_ee_description/meshes/electric_gripper/fingers/extended_wide.DAE" />
+          <mesh filename="file://$(find rethink_ee_description)/meshes/electric_gripper/fingers/extended_wide.DAE" />
         </geometry>
       </visual>

File: rethink_ee_description/urdf/electric_gripper/fingers/half_round_tip.xacro (robot description, xacro)
@@ -10,5 +10,5 @@
         <origin rpy="0 0 ${pi*(g_reflect+1)/2}" xyz="0 0 0"/>
         <geometry>
-          <mesh filename="package://rethink_ee_description/meshes/electric_gripper/fingers/half_round_tip.DAE" />
+          <mesh filename="file://$(find rethink_ee_description)/meshes/electric_gripper/fingers/half_round_tip.DAE" />
         </geometry>
       </visual>

File: rethink_ee_description/urdf/electric_gripper/fingers/paddle_tip.xacro (robot description, xacro)
@@ -10,5 +10,5 @@
         <origin rpy="0 0 ${pi*(g_reflect+1)/2}" xyz="0 0 0"/>
         <geometry>
-          <mesh filename="package://rethink_ee_description/meshes/electric_gripper/fingers/paddle_tip.DAE" />
+          <mesh filename="file://$(find rethink_ee_description)/meshes/electric_gripper/fingers/paddle_tip.DAE" />
         </geometry>
       </visual>

File: rethink_ee_description/urdf/electric_gripper/fingers/standard_narrow.xacro (robot description, xacro)
@@ -8,5 +8,5 @@
         <origin rpy="0 0 ${-pi/2*(reflect+1)}" xyz="0 0 0"/>
         <geometry>
-          <mesh filename="package://rethink_ee_description/meshes/electric_gripper/fingers/standard_narrow.DAE" />
+          <mesh filename="file://$(find rethink_ee_description)/meshes/electric_gripper/fingers/standard_narrow.DAE" />
         </geometry>
       </visual>

File: rethink_ee_description/urdf/electric_gripper/fingers/standard_wide.xacro (robot description, xacro)
@@ -8,5 +8,5 @@
         <origin rpy="0 0 ${-pi/2*(reflect+1)}" xyz="0 0 0"/>
         <geometry>
-          <mesh filename="package://rethink_ee_description/meshes/electric_gripper/fingers/standard_wide.DAE" />
+          <mesh filename="file://$(find rethink_ee_description)/meshes/electric_gripper/fingers/standard_wide.DAE" />
         </geometry>
       </visual>

File: rethink_ee_description/urdf/electric_gripper/rethink_electric_gripper.xacro (robot description, xacro)
@@ -38,5 +38,5 @@
     </xacro:if>
     <!-- Electric Gripper Base Joint -->
-    <joint name="${side}_gripper_base" type="fixed">
+    <joint name="${side}_gripper_base_fixed" type="fixed">
       <origin rpy="0 0 0" xyz="0 0 0.025"/>
       <parent link="${side}_hand"/>

File: rethink_ee_description/urdf/null_gripper/null_gripper.xacro (robot description, xacro)
@@ -19,5 +19,5 @@
     </inertial>
   </link>
-  <joint name="${side}_gripper_base" type="fixed">
+  <joint name="${side}_gripper_base_fixed" type="fixed">
     <origin rpy="0 0 0" xyz="0 0 0"/>
     <parent link="${side}_hand"/>

File: rethink_ee_description/urdf/pneumatic_gripper/pneumatic_gripper_base.xacro (robot description, xacro)
@@ -8,5 +8,5 @@
         <origin rpy="0 ${pi} ${pi}" xyz="0 0 0"/>
         <geometry>
-          <mesh filename="package://rethink_ee_description/meshes/pneumatic_gripper/pneumatic_gripper_base.DAE"/>
+          <mesh filename="file://$(find rethink_ee_description)/meshes/pneumatic_gripper/pneumatic_gripper_base.DAE"/>
         </geometry>
       </visual>
@@ -28,5 +28,5 @@
     </link>
     <!-- Pneumatic Gripper Base Joint -->
-    <joint name="${side}_gripper_base" type="fixed">
+    <joint name="${side}_gripper_base_fixed" type="fixed">
       <origin rpy="0 0 0" xyz="0 0 0.0"/>
       <parent link="${side}_hand"/>

File: rethink_ee_description/urdf/pneumatic_gripper/rethink_pneumatic_gripper.xacro (robot description, xacro)
@@ -8,5 +8,5 @@
         <origin rpy="0 ${pi} ${pi}" xyz="0 0 0"/>
         <geometry>
-          <mesh filename="package://rethink_ee_description/meshes/pneumatic_gripper/pneumatic_gripper_w_cup.DAE"/>
+          <mesh filename="file://$(find rethink_ee_description)/meshes/pneumatic_gripper/pneumatic_gripper_w_cup.DAE"/>
         </geometry>
       </visual>
@@ -27,5 +27,5 @@
     </link>
     <!-- Pneumatic Gripper Base Joint -->
-    <joint name="${side}_gripper_base" type="fixed">
+    <joint name="${side}_gripper_base_fixed" type="fixed">
       <origin rpy="0 0 0" xyz="0 0 0.0"/>
       <parent link="${side}_hand"/>
