Commit message: increase joint efforts

File: baxter_description/urdf/baxter_base/baxter_base.urdf.xacro (robot description, xacro)
@@ -46,5 +46,5 @@
       <origin rpy="0 0 0" xyz="0 0 0"/>
       <geometry>
-        <mesh filename="file://$(find baxter_description)/meshes/torso/base_link.DAE"/>
+        <mesh filename="package://baxter_description/meshes/torso/base_link.DAE"/>
       </geometry>
       <material name="darkgray">
@@ -55,5 +55,5 @@
       <origin rpy="0 0 0" xyz="0 0 0"/>
       <geometry>
-        <mesh filename="file://$(find baxter_description)/meshes/torso/base_link_collision.DAE"/>
+        <mesh filename="package://baxter_description/meshes/torso/base_link_collision.DAE"/>
       </geometry>
     </collision>
@@ -82,5 +82,5 @@
       <origin rpy="0 0 0" xyz="0 0 .00953"/>
       <geometry>
-        <mesh filename="file://$(find baxter_description)/meshes/head/H0.DAE"/>
+        <mesh filename="package://baxter_description/meshes/head/H0.DAE"/>
       </geometry>
       <material name="darkgray">
@@ -126,5 +126,5 @@
       <origin rpy="0 -1.57079632679 0" xyz="0 -.00953 -.0347"/>
       <geometry>
-        <mesh filename="file://$(find baxter_description)/meshes/head/H1.DAE"/>
+        <mesh filename="package://baxter_description/meshes/head/H1.DAE"/>
       </geometry>
       <material name="darkred">
@@ -290,5 +290,5 @@
       <origin rpy="0 0 0" xyz="0 0 0"/>
       <geometry>
-        <mesh filename="file://$(find baxter_description)/meshes/upper_shoulder/S0.DAE"/>
+        <mesh filename="package://baxter_description/meshes/upper_shoulder/S0.DAE"/>
       </geometry>
       <material name="darkred">
@@ -312,5 +312,5 @@
       <origin rpy="0 0 0" xyz="0 0 0"/>
       <geometry>
-        <mesh filename="file://$(find baxter_description)/meshes/lower_shoulder/S1.DAE"/>
+        <mesh filename="package://baxter_description/meshes/lower_shoulder/S1.DAE"/>
       </geometry>
       <material name="darkred">
@@ -334,5 +334,5 @@
       <origin rpy="0 0 0" xyz="0 0 0"/>
       <geometry>
-        <mesh filename="file://$(find baxter_description)/meshes/upper_elbow/E0.DAE"/>
+        <mesh filename="package://baxter_description/meshes/upper_elbow/E0.DAE"/>
       </geometry>
       <material name="darkred">
@@ -369,5 +369,5 @@
       <origin rpy="0 0 0" xyz="0 0 0"/>
       <geometry>
-        <mesh filename="file://$(find baxter_description)/meshes/lower_elbow/E1.DAE"/>
+        <mesh filename="package://baxter_description/meshes/lower_elbow/E1.DAE"/>
       </geometry>
       <material name="darkred">
@@ -391,5 +391,5 @@
       <origin rpy="0 0 0" xyz="0 0 0"/>
       <geometry>
-        <mesh filename="file://$(find baxter_description)/meshes/upper_forearm/W0.DAE"/>
+        <mesh filename="package://baxter_description/meshes/upper_forearm/W0.DAE"/>
       </geometry>
       <material name="darkred">
@@ -433,5 +433,5 @@
       <origin rpy="0 0 0" xyz="0 0 0"/>
       <geometry>
-        <mesh filename="file://$(find baxter_description)/meshes/lower_forearm/W1.DAE"/>
+        <mesh filename="package://baxter_description/meshes/lower_forearm/W1.DAE"/>
       </geometry>
       <material name="darkred">
@@ -455,5 +455,5 @@
       <origin rpy="0 0 0" xyz="0 0 0"/>
       <geometry>
-        <mesh filename="file://$(find baxter_description)/meshes/wrist/W2.DAE"/>
+        <mesh filename="package://baxter_description/meshes/wrist/W2.DAE"/>
       </geometry>
       <material name="lightgrey">
@@ -552,5 +552,5 @@
     <parent link="right_arm_mount"/>
     <child link="right_upper_shoulder"/>
-    <limit effort="50.0" lower="-1.70167993878" upper="1.70167993878" velocity="1.5"/>
+    <limit effort="100.0" lower="-1.70167993878" upper="1.70167993878" velocity="1.5"/>
     <dynamics damping="0.7" friction="0.0"/>
   </joint>
@@ -560,5 +560,5 @@
     <parent link="right_upper_shoulder"/>
     <child link="right_lower_shoulder"/>
-    <limit effort="50.0" lower="-2.147" upper="1.047" velocity="1.5"/>
+    <limit effort="100.0" lower="-2.147" upper="1.047" velocity="1.5"/>
     <dynamics damping="0.7" friction="0.0"/>
   </joint>
@@ -568,5 +568,5 @@
     <parent link="right_lower_shoulder"/>
     <child link="right_upper_elbow"/>
-    <limit effort="50.0" lower="-3.05417993878" upper="3.05417993878" velocity="1.5"/>
+    <limit effort="100.0" lower="-3.05417993878" upper="3.05417993878" velocity="1.5"/>
     <dynamics damping="0.7" friction="0.0"/>
   </joint>
@@ -582,5 +582,5 @@
     <parent link="right_upper_elbow"/>
     <child link="right_lower_elbow"/>
-    <limit effort="50.0" lower="-0.05" upper="2.618" velocity="1.5"/>
+    <limit effort="100.0" lower="-0.05" upper="2.618" velocity="1.5"/>
     <dynamics damping="0.7" friction="0.0"/>
   </joint>
@@ -590,5 +590,5 @@
     <parent link="right_lower_elbow"/>
     <child link="right_upper_forearm"/>
-    <limit effort="15.0" lower="-3.059" upper="3.059" velocity="4.0"/>
+    <limit effort="50.0" lower="-3.059" upper="3.059" velocity="4.0"/>
     <dynamics damping="0.7" friction="0.0"/>
   </joint>
@@ -610,5 +610,5 @@
     <parent link="right_upper_forearm"/>
     <child link="right_lower_forearm"/>
-    <limit effort="15.0" lower="-1.57079632679" upper="2.094" velocity="4.0"/>
+    <limit effort="50.0" lower="-1.57079632679" upper="2.094" velocity="4.0"/>
     <dynamics damping="0.7" friction="0.0"/>
   </joint>
@@ -618,5 +618,5 @@
     <parent link="right_lower_forearm"/>
     <child link="right_wrist"/>
-    <limit effort="15.0" lower="-3.059" upper="3.059" velocity="4.0"/>
+    <limit effort="50.0" lower="-3.059" upper="3.059" velocity="4.0"/>
     <dynamics damping="0.7" friction="0.0"/>
   </joint>
@@ -659,5 +659,5 @@
       <origin rpy="0 0 0" xyz="0 0 0"/>
       <geometry>
-        <mesh filename="file://$(find baxter_description)/meshes/upper_shoulder/S0.DAE"/>
+        <mesh filename="package://baxter_description/meshes/upper_shoulder/S0.DAE"/>
       </geometry>
       <material name="darkred">
@@ -681,5 +681,5 @@
       <origin rpy="0 0 0" xyz="0 0 0"/>
       <geometry>
-        <mesh filename="file://$(find baxter_description)/meshes/lower_shoulder/S1.DAE"/>
+        <mesh filename="package://baxter_description/meshes/lower_shoulder/S1.DAE"/>
       </geometry>
       <material name="darkred">
@@ -703,5 +703,5 @@
       <origin rpy="0 0 0" xyz="0 0 0"/>
       <geometry>
-        <mesh filename="file://$(find baxter_description)/meshes/upper_elbow/E0.DAE"/>
+        <mesh filename="package://baxter_description/meshes/upper_elbow/E0.DAE"/>
       </geometry>
       <material name="darkred">
@@ -738,5 +738,5 @@
       <origin rpy="0 0 0" xyz="0 0 0"/>
       <geometry>
-        <mesh filename="file://$(find baxter_description)/meshes/lower_elbow/E1.DAE"/>
+        <mesh filename="package://baxter_description/meshes/lower_elbow/E1.DAE"/>
       </geometry>
       <material name="darkred">
@@ -760,5 +760,5 @@
       <origin rpy="0 0 0" xyz="0 0 0"/>
       <geometry>
-        <mesh filename="file://$(find baxter_description)/meshes/upper_forearm/W0.DAE"/>
+        <mesh filename="package://baxter_description/meshes/upper_forearm/W0.DAE"/>
       </geometry>
       <material name="darkred">
@@ -802,5 +802,5 @@
       <origin rpy="0 0 0" xyz="0 0 0"/>
       <geometry>
-        <mesh filename="file://$(find baxter_description)/meshes/lower_forearm/W1.DAE"/>
+        <mesh filename="package://baxter_description/meshes/lower_forearm/W1.DAE"/>
       </geometry>
       <material name="darkred">
@@ -824,5 +824,5 @@
       <origin rpy="0 0 0" xyz="0 0 0"/>
       <geometry>
-        <mesh filename="file://$(find baxter_description)/meshes/wrist/W2.DAE"/>
+        <mesh filename="package://baxter_description/meshes/wrist/W2.DAE"/>
       </geometry>
       <material name="lightgrey">
@@ -921,5 +921,5 @@
     <parent link="left_arm_mount"/>
     <child link="left_upper_shoulder"/>
-    <limit effort="50.0" lower="-1.70167993878" upper="1.70167993878" velocity="1.5"/>
+    <limit effort="100.0" lower="-1.70167993878" upper="1.70167993878" velocity="1.5"/>
     <dynamics damping="0.7" friction="0.0"/>
   </joint>
@@ -929,5 +929,5 @@
     <parent link="left_upper_shoulder"/>
     <child link="left_lower_shoulder"/>
-    <limit effort="50.0" lower="-2.147" upper="1.047" velocity="1.5"/>
+    <limit effort="100.0" lower="-2.147" upper="1.047" velocity="1.5"/>
     <dynamics damping="0.7" friction="0.0"/>
   </joint>
@@ -937,5 +937,5 @@
     <parent link="left_lower_shoulder"/>
     <child link="left_upper_elbow"/>
-    <limit effort="50.0" lower="-3.05417993878" upper="3.05417993878" velocity="1.5"/>
+    <limit effort="100.0" lower="-3.05417993878" upper="3.05417993878" velocity="1.5"/>
     <dynamics damping="0.7" friction="0.0"/>
   </joint>
@@ -951,5 +951,5 @@
     <parent link="left_upper_elbow"/>
     <child link="left_lower_elbow"/>
-    <limit effort="50.0" lower="-0.05" upper="2.618" velocity="1.5"/>
+    <limit effort="100.0" lower="-0.05" upper="2.618" velocity="1.5"/>
     <dynamics damping="0.7" friction="0.0"/>
   </joint>
@@ -959,5 +959,5 @@
     <parent link="left_lower_elbow"/>
     <child link="left_upper_forearm"/>
-    <limit effort="15.0" lower="-3.059" upper="3.059" velocity="4.0"/>
+    <limit effort="50.0" lower="-3.059" upper="3.059" velocity="4.0"/>
     <dynamics damping="0.7" friction="0.0"/>
   </joint>
@@ -979,5 +979,5 @@
     <parent link="left_upper_forearm"/>
     <child link="left_lower_forearm"/>
-    <limit effort="15.0" lower="-1.57079632679" upper="2.094" velocity="4.0"/>
+    <limit effort="50.0" lower="-1.57079632679" upper="2.094" velocity="4.0"/>
     <dynamics damping="0.7" friction="0.0"/>
   </joint>
@@ -987,5 +987,5 @@
     <parent link="left_lower_forearm"/>
     <child link="left_wrist"/>
-    <limit effort="15.0" lower="-3.059" upper="3.059" velocity="4.0"/>
+    <limit effort="50.0" lower="-3.059" upper="3.059" velocity="4.0"/>
     <dynamics damping="0.7" friction="0.0"/>
   </joint>
